Commit message: completed the basic urdf model

File: body.urdf (robot description, URDF)
Before this commit: robot Krever, 6 links, 5 joints
Links:
- removed link caster_wheel
- added link caster_wheel1; collision sphere radius=0.05; visual sphere radius=0.05
- added link caster_wheel2; collision sphere radius=0.05; visual sphere radius=0.05
- added link support_rod; collision box size=0.1 0.1 1.07; visual box size=0.1 0.1 1.07
- added link tray; collision box size=0.65 0.8 0.01; visual box size=0.65 0.8 0.01
- added link u1; collision box size=0.6 0.1 0.04; visual box size=0.6 0.1 0.04
- added link u2; collision box size=0.6 0.1 0.04; visual box size=0.6 0.1 0.04
- added link u3; collision box size=0.6 0.1 0.04; visual box size=0.6 0.1 0.04
- link base_link: geometry collision box size=0.6 0.8 0.3; visual box size=0.8 0.6 0.3
- link left_wheel: geometry collision cylinder length=0.05 radius=0.1; visual cylinder length=0.05 radius=0.1
- link lidar: geometry collision cylinder length=0.05 radius=0.1; visual cylinder length=0.05 radius=0.1
- link right_wheel: geometry collision cylinder length=0.05 radius=0.1; visual cylinder length=0.05 radius=0.1
Joints:
- removed joint body_caster_wheel_joint
- added joint base_suppot_joint: type fixed, parent base_link, child support_rod, origin xyz=-0.35 0. 0.835 rpy=0.0 0.0 0.0, limit lower=0.0 upper=0.0 effort=0.0 velocity=0.0
- added joint body_caster_wheel_joint1: type fixed, parent base_link, child caster_wheel1, origin xyz=0.3 0 -0.05 rpy=0 0 0
- added joint body_caster_wheel_joint2: type fixed, parent base_link, child caster_wheel2, origin xyz=-0.3 0 -0.05 rpy=0 0 0
- added joint joint_name: type fixed, parent support_rod, child tray, origin xyz=0.375 0.0 -0.465 rpy=0.0 0.0 0.0, limit lower=0.0 upper=0.0 effort=0.0 velocity=0.0
- added joint u1: type fixed, parent support_rod, child u1, origin xyz=0 0 0.555 rpy=0.0 0.0 1.57, limit lower=0.0 upper=0.0 effort=0.0 velocity=0.0
- added joint u2: type fixed, parent support_rod, child u2, origin xyz=0.25 0.35 0.555 rpy=0.0 0.0 0, limit lower=0.0 upper=0.0 effort=0.0 velocity=0.0
- added joint u3: type fixed, parent support_rod, child u3, origin xyz=0.25 -0.35 0.555 rpy=0.0 0.0 0, limit lower=0.0 upper=0.0 effort=0.0 velocity=0.0
- joint base_left_wheel_joint: origin xyz=-0.15 0.325 0 rpy=0 0 0 -> xyz=0 0.325 0 rpy=0 0 0
- joint base_right_wheel_joint: origin xyz=-0.15 -0.325 0 rpy=0 0 0 -> xyz=-0 -0.325 0 rpy=0 0 0
